Commit message: Add dummy link for inertia

File: fetch_description/robots/fetch.urdf (robot description, URDF)
Before this commit: robot fetch, 26 links, 25 joints
Links:
- added link inertial_base_link, mass 70.1294
- link base_link: mass 70.1294 -> None
Joints:
- added joint base_inertial_joint: type fixed, parent base_link, child inertial_base_link, origin xyz=0 0 0 rpy=0 0 0, axis 0 1 0
